Commit message: 1

File: robot/H1_2/urdf/h1_2.urdf (robot description, URDF)
Before this commit: robot h1_2, 75 links, 74 joints
Links:
- link L_hand_base_link: geometry collision mesh filename=../../H1_2/meshes/L_hand_base_link.STL; visual mesh filename=../../H1_2/meshes/L_hand_base_link.STL
- link L_index_intermediate: geometry collision mesh filename=../../H1_2/meshes/link16_L.STL; visual mesh filename=../../H1_2/meshes/link16_L.STL
- link L_index_proximal: geometry collision mesh filename=../../H1_2/meshes/link15_L.STL; visual mesh filename=../../H1_2/meshes/link15_L.STL
- link L_middle_intermediate: geometry collision mesh filename=../../H1_2/meshes/link18_L.STL; visual mesh filename=../../H1_2/meshes/link18_L.STL
- link L_middle_proximal: geometry collision mesh filename=../../H1_2/meshes/link17_L.STL; visual mesh filename=../../H1_2/meshes/link17_L.STL
- link L_pinky_intermediate: geometry collision mesh filename=../../H1_2/meshes/link22_L.STL; visual mesh filename=../../H1_2/meshes/link22_L.STL
- link L_pinky_proximal: geometry collision mesh filename=../../H1_2/meshes/link21_L.STL; visual mesh filename=../../H1_2/meshes/link21_L.STL
- link L_ring_intermediate: geometry collision mesh filename=../../H1_2/meshes/link20_L.STL; visual mesh filename=../../H1_2/meshes/link20_L.STL
- link L_ring_proximal: geometry collision mesh filename=../../H1_2/meshes/link19_L.STL; visual mesh filename=../../H1_2/meshes/link19_L.STL
- link L_thumb_distal: geometry collision mesh filename=../../H1_2/meshes/link14_L.STL; visual mesh filename=../../H1_2/meshes/link14_L.STL
- link L_thumb_intermediate: geometry collision mesh filename=../../H1_2/meshes/link13_L.STL; visual mesh filename=../../H1_2/meshes/link13_L.STL
- link L_thumb_proximal: geometry collision mesh filename=../../H1_2/meshes/link12_L.STL; visual mesh filename=../../H1_2/meshes/link12_L.STL
- link L_thumb_proximal_base: geometry collision mesh filename=../../H1_2/meshes/link11_L.STL; visual mesh filename=../../H1_2/meshes/link11_L.STL
- link R_hand_base_link: geometry collision mesh filename=../../H1_2/meshes/R_hand_base_link.STL; visual mesh filename=../../H1_2/meshes/R_hand_base_link.STL
- link R_index_intermediate: geometry collision mesh filename=../../H1_2/meshes/link16_R.STL; visual mesh filename=../../H1_2/meshes/link16_R.STL
- link R_index_proximal: geometry collision mesh filename=../../H1_2/meshes/link15_R.STL; visual mesh filename=../../H1_2/meshes/link15_R.STL
- link R_middle_intermediate: geometry collision mesh filename=../../H1_2/meshes/link18_R.STL; visual mesh filename=../../H1_2/meshes/link18_R.STL
- link R_middle_proximal: geometry collision mesh filename=../../H1_2/meshes/link17_R.STL; visual mesh filename=../../H1_2/meshes/link17_R.STL
- link R_pinky_intermediate: geometry collision mesh filename=../../H1_2/meshes/link22_R.STL; visual mesh filename=../../H1_2/meshes/link22_R.STL
- link R_pinky_proximal: geometry collision mesh filename=../../H1_2/meshes/link21_R.STL; visual mesh filename=../../H1_2/meshes/link21_R.STL
- link R_ring_intermediate: geometry collision mesh filename=../../H1_2/meshes/link20_R.STL; visual mesh filename=../../H1_2/meshes/link20_R.STL
- link R_ring_proximal: geometry collision mesh filename=../../H1_2/meshes/link19_R.STL; visual mesh filename=../../H1_2/meshes/link19_R.STL
- link R_thumb_distal: geometry collision mesh filename=../../H1_2/meshes/link14_R.STL; visual mesh filename=../../H1_2/meshes/link14_R.STL
- link R_thumb_intermediate: geometry collision mesh filename=../../H1_2/meshes/link13_R.STL; visual mesh filename=../../H1_2/meshes/link13_R.STL
- link R_thumb_proximal: geometry collision mesh filename=../../H1_2/meshes/link12_R.STL; visual mesh filename=../../H1_2/meshes/link12_R.STL
- link R_thumb_proximal_base: geometry collision mesh filename=../../H1_2/meshes/link11_R.STL; visual mesh filename=../../H1_2/meshes/link11_R.STL
- link left_ankle_pitch_link: geometry collision mesh filename=../../H1_2/meshes/left_ankle_pitch_link.STL; visual mesh filename=../../H1_2/meshes/left_ankle_pitch_link.STL
- link left_ankle_roll_link: geometry collision mesh filename=../../H1_2/meshes/left_ankle_roll_link.STL; visual mesh filename=../../H1_2/meshes/left_ankle_roll_link.STL
- link left_elbow_link: geometry collision mesh filename=../../H1_2/meshes/left_elbow_link.STL; visual mesh filename=../../H1_2/meshes/left_elbow_link.STL
- link left_hip_pitch_link: geometry collision cylinder length=0.2 radius=0.02; visual mesh filename=../../H1_2/meshes/left_hip_pitch_link.STL
- link left_hip_roll_link: geometry collision cylinder length=0.01 radius=0.02; visual mesh filename=../../H1_2/meshes/left_hip_roll_link.STL
- link left_hip_yaw_link: geometry collision cylinder length=0.02 radius=0.01; visual mesh filename=../../H1_2/meshes/left_hip_yaw_link.STL
- link left_knee_link: geometry collision cylinder length=0.2 radius=0.02; visual mesh filename=../../H1_2/meshes/left_knee_link.STL
- link left_shoulder_pitch_link: geometry collision mesh filename=../../H1_2/meshes/left_shoulder_pitch_link.STL; visual mesh filename=../../H1_2/meshes/left_shoulder_pitch_link.STL
- link left_shoulder_roll_link: geometry collision mesh filename=../../H1_2/meshes/left_shoulder_roll_link.STL; visual mesh filename=../../H1_2/meshes/left_shoulder_roll_link.STL
- link left_shoulder_yaw_link: geometry collision mesh filename=../../H1_2/meshes/left_shoulder_yaw_link.STL; visual mesh filename=../../H1_2/meshes/left_shoulder_yaw_link.STL
- link left_wrist_pitch_link: geometry collision mesh filename=../../H1_2/meshes/left_wrist_pitch_link.STL; visual mesh filename=../../H1_2/meshes/left_wrist_pitch_link.STL
- link left_wrist_roll_link: geometry collision mesh filename=../../H1_2/meshes/left_wrist_roll_link.STL; visual mesh filename=../../H1_2/meshes/left_wrist_roll_link.STL
- link left_wrist_yaw_link: geometry visual mesh filename=../../H1_2/meshes/wrist_yaw_link.STL
- link logo_link: geometry visual mesh filename=../../H1_2/meshes/logo_link.STL
- link pelvis: geometry collision sphere radius=0.05; visual mesh filename=../../H1_2/meshes/pelvis.STL
- link right_ankle_pitch_link: geometry collision mesh filename=../../H1_2/meshes/right_ankle_pitch_link.STL; visual mesh filename=../../H1_2/meshes/right_ankle_pitch_link.STL
- link right_ankle_roll_link: geometry collision mesh filename=../../H1_2/meshes/right_ankle_roll_link.STL; visual mesh filename=../../H1_2/meshes/right_ankle_roll_link.STL
- link right_elbow_link: geometry collision mesh filename=../../H1_2/meshes/right_elbow_link.STL; visual mesh filename=../../H1_2/meshes/right_elbow_link.STL
- link right_hip_pitch_link: geometry collision cylinder length=0.2 radius=0.02; visual mesh filename=../../H1_2/meshes/right_hip_pitch_link.STL
- link right_hip_roll_link: geometry collision cylinder length=0.01 radius=0.02; visual mesh filename=../../H1_2/meshes/right_hip_roll_link.STL
- link right_hip_yaw_link: geometry collision cylinder length=0.02 radius=0.01; visual mesh filename=../../H1_2/meshes/right_hip_yaw_link.STL
- link right_knee_link: geometry collision cylinder length=0.2 radius=0.02; visual mesh filename=../../H1_2/meshes/right_knee_link.STL
- link right_shoulder_pitch_link: geometry collision mesh filename=../../H1_2/meshes/right_shoulder_pitch_link.STL; visual mesh filename=../../H1_2/meshes/right_shoulder_pitch_link.STL
- link right_shoulder_roll_link: geometry collision mesh filename=../../H1_2/meshes/right_shoulder_roll_link.STL; visual mesh filename=../../H1_2/meshes/right_shoulder_roll_link.STL
- link right_shoulder_yaw_link: geometry collision mesh filename=../../H1_2/meshes/right_shoulder_yaw_link.STL; visual mesh filename=../../H1_2/meshes/right_shoulder_yaw_link.STL
- link right_wrist_pitch_link: geometry collision mesh filename=../../H1_2/meshes/right_wrist_pitch_link.STL; visual mesh filename=../../H1_2/meshes/right_wrist_pitch_link.STL
- link right_wrist_roll_link: geometry collision mesh filename=../../H1_2/meshes/right_wrist_roll_link.STL; visual mesh filename=../../H1_2/meshes/right_wrist_roll_link.STL
- link right_wrist_yaw_link: geometry visual mesh filename=../../H1_2/meshes/wrist_yaw_link.STL
- link torso_link: geometry collision box size=0.08 0.16 0.1; visual mesh filename=../../H1_2/meshes/torso_link.STL
