Commit message: bash

File: robot/GR1T2/urdf/gr1t2.urdf (robot description, URDF)
Before this commit: robot ../../GR1T2, 51 links, 50 joints
Links:
- link base: geometry collision mesh filename=GR1T2//meshes/base.STL; visual mesh filename=GR1T2//meshes/base.STL
- link head_pitch: geometry visual mesh filename=GR1T2//meshes/head_pitch.STL
- link head_roll: geometry visual mesh filename=GR1T2//meshes/head_roll.STL
- link head_yaw: geometry collision sphere radius=0.12; visual mesh filename=GR1T2//meshes/head_yaw.STL
- link l_foot_pitch: geometry visual mesh filename=GR1T2//meshes/l_foot_pitch.STL
- link l_foot_roll: geometry collision cylinder length=0.24 radius=0.02; collision cylinder length=0.24 radius=0.02
- link l_hand_pitch: geometry collision box size=0.1 0.05 0.2; visual mesh filename=GR1T2//meshes/l_hand_pitch.STL
- link l_hand_roll: geometry visual mesh filename=GR1T2//meshes/l_hand_roll.STL
- link l_hand_yaw: geometry collision box size=0.065 0.065 0.2; visual mesh filename=GR1T2//meshes/l_hand_yaw.STL
- link l_lower_arm_pitch: geometry visual mesh filename=GR1T2//meshes/l_lower_arm_pitch.STL
- link l_shank_pitch: geometry collision box size=0.07 0.07 0.28; visual mesh filename=GR1T2//meshes/l_shank_pitch.STL
- link l_thigh_pitch: geometry collision box size=0.12 0.08 0.2; collision cylinder length=0.08 radius=0.1
- link l_thigh_roll: geometry visual mesh filename=GR1T2//meshes/l_thigh_roll.STL
- link l_thigh_yaw: geometry collision mesh filename=GR1T2//meshes/l_thigh_yaw.STL; visual mesh filename=GR1T2//meshes/l_thigh_yaw.STL
- link l_upper_arm_pitch: geometry visual mesh filename=GR1T2//meshes/l_upper_arm_pitch.STL
- link l_upper_arm_roll: geometry collision cylinder length=0.08 radius=0.04; visual mesh filename=GR1T2//meshes/l_upper_arm_roll.STL
- link l_upper_arm_yaw: geometry collision cylinder length=0.14 radius=0.035; visual mesh filename=GR1T2//meshes/l_upper_arm_yaw.STL
- link r_foot_pitch: geometry visual mesh filename=GR1T2//meshes/r_foot_pitch.STL
- link r_foot_roll: geometry collision cylinder length=0.24 radius=0.02; collision cylinder length=0.24 radius=0.02
- link r_hand_pitch: geometry collision box size=0.1 0.05 0.2; visual mesh filename=GR1T2//meshes/r_hand_pitch.STL
- link r_hand_roll: geometry visual mesh filename=GR1T2//meshes/r_hand_roll.STL
- link r_hand_yaw: geometry collision box size=0.065 0.065 0.2; visual mesh filename=GR1T2//meshes/r_hand_yaw.STL
- link r_lower_arm_pitch: geometry visual mesh filename=GR1T2//meshes/r_lower_arm_pitch.STL
- link r_shank_pitch: geometry collision box size=0.07 0.07 0.28; visual mesh filename=GR1T2//meshes/r_shank_pitch.STL
- link r_thigh_pitch: geometry collision box size=0.12 0.08 0.2; collision cylinder length=0.08 radius=0.1
- link r_thigh_roll: geometry visual mesh filename=GR1T2//meshes/r_thigh_roll.STL
- link r_thigh_yaw: geometry collision mesh filename=GR1T2//meshes/r_thigh_yaw.STL; visual mesh filename=GR1T2//meshes/r_thigh_yaw.STL
- link r_upper_arm_pitch: geometry visual mesh filename=GR1T2//meshes/r_upper_arm_pitch.STL
- link r_upper_arm_roll: geometry collision cylinder length=0.08 radius=0.04; visual mesh filename=GR1T2//meshes/r_upper_arm_roll.STL
- link r_upper_arm_yaw: geometry collision cylinder length=0.14 radius=0.035; visual mesh filename=GR1T2//meshes/r_upper_arm_yaw.STL
- link torso: geometry collision mesh filename=GR1T2//meshes/torso.STL; visual mesh filename=GR1T2//meshes/torso.STL
- link waist_pitch: geometry visual mesh filename=GR1T2//meshes/waist_pitch.STL
- link waist_roll: geometry visual mesh filename=GR1T2//meshes/waist_roll.STL
- link waist_yaw: geometry collision mesh filename=GR1T2//meshes/waist_yaw.STL; visual mesh filename=GR1T2//meshes/waist_yaw.STL

File: robot/H1_2/urdf/h1_2.urdf (robot description, URDF)
Before this commit: robot ../../H1_2, 75 links, 74 joints
Links:
- link L_hand_base_link: geometry collision mesh filename=H1_2/meshes/L_hand_base_link.STL; visual mesh filename=H1_2/meshes/L_hand_base_link.STL
- link L_index_intermediate: geometry collision mesh filename=H1_2/meshes/link16_L.STL; visual mesh filename=H1_2/meshes/link16_L.STL
- link L_index_proximal: geometry collision mesh filename=H1_2/meshes/link15_L.STL; visual mesh filename=H1_2/meshes/link15_L.STL
- link L_middle_intermediate: geometry collision mesh filename=H1_2/meshes/link18_L.STL; visual mesh filename=H1_2/meshes/link18_L.STL
- link L_middle_proximal: geometry collision mesh filename=H1_2/meshes/link17_L.STL; visual mesh filename=H1_2/meshes/link17_L.STL
- link L_pinky_intermediate: geometry collision mesh filename=H1_2/meshes/link22_L.STL; visual mesh filename=H1_2/meshes/link22_L.STL
- link L_pinky_proximal: geometry collision mesh filename=H1_2/meshes/link21_L.STL; visual mesh filename=H1_2/meshes/link21_L.STL
- link L_ring_intermediate: geometry collision mesh filename=H1_2/meshes/link20_L.STL; visual mesh filename=H1_2/meshes/link20_L.STL
- link L_ring_proximal: geometry collision mesh filename=H1_2/meshes/link19_L.STL; visual mesh filename=H1_2/meshes/link19_L.STL
- link L_thumb_distal: geometry collision mesh filename=H1_2/meshes/link14_L.STL; visual mesh filename=H1_2/meshes/link14_L.STL
- link L_thumb_intermediate: geometry collision mesh filename=H1_2/meshes/link13_L.STL; visual mesh filename=H1_2/meshes/link13_L.STL
- link L_thumb_proximal: geometry collision mesh filename=H1_2/meshes/link12_L.STL; visual mesh filename=H1_2/meshes/link12_L.STL
- link L_thumb_proximal_base: geometry collision mesh filename=H1_2/meshes/link11_L.STL; visual mesh filename=H1_2/meshes/link11_L.STL
- link R_hand_base_link: geometry collision mesh filename=H1_2/meshes/R_hand_base_link.STL; visual mesh filename=H1_2/meshes/R_hand_base_link.STL
- link R_index_intermediate: geometry collision mesh filename=H1_2/meshes/link16_R.STL; visual mesh filename=H1_2/meshes/link16_R.STL
- link R_index_proximal: geometry collision mesh filename=H1_2/meshes/link15_R.STL; visual mesh filename=H1_2/meshes/link15_R.STL
- link R_middle_intermediate: geometry collision mesh filename=H1_2/meshes/link18_R.STL; visual mesh filename=H1_2/meshes/link18_R.STL
- link R_middle_proximal: geometry collision mesh filename=H1_2/meshes/link17_R.STL; visual mesh filename=H1_2/meshes/link17_R.STL
- link R_pinky_intermediate: geometry collision mesh filename=H1_2/meshes/link22_R.STL; visual mesh filename=H1_2/meshes/link22_R.STL
- link R_pinky_proximal: geometry collision mesh filename=H1_2/meshes/link21_R.STL; visual mesh filename=H1_2/meshes/link21_R.STL
- link R_ring_intermediate: geometry collision mesh filename=H1_2/meshes/link20_R.STL; visual mesh filename=H1_2/meshes/link20_R.STL
- link R_ring_proximal: geometry collision mesh filename=H1_2/meshes/link19_R.STL; visual mesh filename=H1_2/meshes/link19_R.STL
- link R_thumb_distal: geometry collision mesh filename=H1_2/meshes/link14_R.STL; visual mesh filename=H1_2/meshes/link14_R.STL
- link R_thumb_intermediate: geometry collision mesh filename=H1_2/meshes/link13_R.STL; visual mesh filename=H1_2/meshes/link13_R.STL
- link R_thumb_proximal: geometry collision mesh filename=H1_2/meshes/link12_R.STL; visual mesh filename=H1_2/meshes/link12_R.STL
- link R_thumb_proximal_base: geometry collision mesh filename=H1_2/meshes/link11_R.STL; visual mesh filename=H1_2/meshes/link11_R.STL
- link left_ankle_pitch_link: geometry collision mesh filename=H1_2/meshes/left_ankle_pitch_link.STL; visual mesh filename=H1_2/meshes/left_ankle_pitch_link.STL
- link left_ankle_roll_link: geometry collision mesh filename=H1_2/meshes/left_ankle_roll_link.STL; visual mesh filename=H1_2/meshes/left_ankle_roll_link.STL
- link left_elbow_link: geometry collision mesh filename=H1_2/meshes/left_elbow_link.STL; visual mesh filename=H1_2/meshes/left_elbow_link.STL
- link left_hip_pitch_link: geometry collision cylinder length=0.2 radius=0.02; visual mesh filename=H1_2/meshes/left_hip_pitch_link.STL
- link left_hip_roll_link: geometry collision cylinder length=0.01 radius=0.02; visual mesh filename=H1_2/meshes/left_hip_roll_link.STL
- link left_hip_yaw_link: geometry collision cylinder length=0.02 radius=0.01; visual mesh filename=H1_2/meshes/left_hip_yaw_link.STL
- link left_knee_link: geometry collision cylinder length=0.2 radius=0.02; visual mesh filename=H1_2/meshes/left_knee_link.STL
- link left_shoulder_pitch_link: geometry collision mesh filename=H1_2/meshes/left_shoulder_pitch_link.STL; visual mesh filename=H1_2/meshes/left_shoulder_pitch_link.STL
- link left_shoulder_roll_link: geometry collision mesh filename=H1_2/meshes/left_shoulder_roll_link.STL; visual mesh filename=H1_2/meshes/left_shoulder_roll_link.STL
- link left_shoulder_yaw_link: geometry collision mesh filename=H1_2/meshes/left_shoulder_yaw_link.STL; visual mesh filename=H1_2/meshes/left_shoulder_yaw_link.STL
- link left_wrist_pitch_link: geometry collision mesh filename=H1_2/meshes/left_wrist_pitch_link.STL; visual mesh filename=H1_2/meshes/left_wrist_pitch_link.STL
- link left_wrist_roll_link: geometry collision mesh filename=H1_2/meshes/left_wrist_roll_link.STL; visual mesh filename=H1_2/meshes/left_wrist_roll_link.STL
- link left_wrist_yaw_link: geometry visual mesh filename=H1_2/meshes/wrist_yaw_link.STL
- link logo_link: geometry visual mesh filename=H1_2/meshes/logo_link.STL
- link pelvis: geometry collision sphere radius=0.05; visual mesh filename=H1_2/meshes/pelvis.STL
- link right_ankle_pitch_link: geometry collision mesh filename=H1_2/meshes/right_ankle_pitch_link.STL; visual mesh filename=H1_2/meshes/right_ankle_pitch_link.STL
- link right_ankle_roll_link: geometry collision mesh filename=H1_2/meshes/right_ankle_roll_link.STL; visual mesh filename=H1_2/meshes/right_ankle_roll_link.STL
- link right_elbow_link: geometry collision mesh filename=H1_2/meshes/right_elbow_link.STL; visual mesh filename=H1_2/meshes/right_elbow_link.STL
- link right_hip_pitch_link: geometry collision cylinder length=0.2 radius=0.02; visual mesh filename=H1_2/meshes/right_hip_pitch_link.STL
- link right_hip_roll_link: geometry collision cylinder length=0.01 radius=0.02; visual mesh filename=H1_2/meshes/right_hip_roll_link.STL
- link right_hip_yaw_link: geometry collision cylinder length=0.02 radius=0.01; visual mesh filename=H1_2/meshes/right_hip_yaw_link.STL
- link right_knee_link: geometry collision cylinder length=0.2 radius=0.02; visual mesh filename=H1_2/meshes/right_knee_link.STL
- link right_shoulder_pitch_link: geometry collision mesh filename=H1_2/meshes/right_shoulder_pitch_link.STL; visual mesh filename=H1_2/meshes/right_shoulder_pitch_link.STL
- link right_shoulder_roll_link: geometry collision mesh filename=H1_2/meshes/right_shoulder_roll_link.STL; visual mesh filename=H1_2/meshes/right_shoulder_roll_link.STL
- link right_shoulder_yaw_link: geometry collision mesh filename=H1_2/meshes/right_shoulder_yaw_link.STL; visual mesh filename=H1_2/meshes/right_shoulder_yaw_link.STL
- link right_wrist_pitch_link: geometry collision mesh filename=H1_2/meshes/right_wrist_pitch_link.STL; visual mesh filename=H1_2/meshes/right_wrist_pitch_link.STL
- link right_wrist_roll_link: geometry collision mesh filename=H1_2/meshes/right_wrist_roll_link.STL; visual mesh filename=H1_2/meshes/right_wrist_roll_link.STL
- link right_wrist_yaw_link: geometry visual mesh filename=H1_2/meshes/wrist_yaw_link.STL
- link torso_link: geometry collision box size=0.08 0.16 0.1; visual mesh filename=H1_2/meshes/torso_link.STL

Commit message: 1

File: robot/GR1T2/urdf/gr1t2.urdf (robot description, URDF)
Before this commit: robot GR1T2/meshes, 51 links, 50 joints
Links:
- link base: geometry collision mesh filename=GR1T2/meshes/base.STL; visual mesh filename=GR1T2/meshes/base.STL
- link head_pitch: geometry visual mesh filename=GR1T2/meshes/head_pitch.STL
- link head_roll: geometry visual mesh filename=GR1T2/meshes/head_roll.STL
- link head_yaw: geometry collision sphere radius=0.12; visual mesh filename=GR1T2/meshes/head_yaw.STL
- link keyframe_left_collar_link: geometry visual sphere radius=0.05
- link l_foot_pitch: geometry visual mesh filename=GR1T2/meshes/l_foot_pitch.STL
- link l_foot_roll: geometry collision cylinder length=0.24 radius=0.02; collision cylinder length=0.24 radius=0.02
- link l_hand_pitch: geometry collision box size=0.1 0.05 0.2; visual mesh filename=GR1T2/meshes/l_hand_pitch.STL
- link l_hand_roll: geometry visual mesh filename=GR1T2/meshes/l_hand_roll.STL
- link l_hand_yaw: geometry collision box size=0.065 0.065 0.2; visual mesh filename=GR1T2/meshes/l_hand_yaw.STL
- link l_lower_arm_pitch: geometry visual mesh filename=GR1T2/meshes/l_lower_arm_pitch.STL
- link l_shank_pitch: geometry collision box size=0.07 0.07 0.28; visual mesh filename=GR1T2/meshes/l_shank_pitch.STL
- link l_thigh_pitch: geometry collision box size=0.12 0.08 0.2; collision cylinder length=0.08 radius=0.1
- link l_thigh_roll: geometry visual mesh filename=GR1T2/meshes/l_thigh_roll.STL
- link l_thigh_yaw: geometry collision mesh filename=GR1T2/meshes/l_thigh_yaw.STL; visual mesh filename=GR1T2/meshes/l_thigh_yaw.STL
- link l_upper_arm_pitch: geometry visual mesh filename=GR1T2/meshes/l_upper_arm_pitch.STL
- link l_upper_arm_roll: geometry collision cylinder length=0.08 radius=0.04; visual mesh filename=GR1T2/meshes/l_upper_arm_roll.STL
- link l_upper_arm_yaw: geometry collision cylinder length=0.14 radius=0.035; visual mesh filename=GR1T2/meshes/l_upper_arm_yaw.STL
- link r_foot_pitch: geometry visual mesh filename=GR1T2/meshes/r_foot_pitch.STL
- link r_foot_roll: geometry collision cylinder length=0.24 radius=0.02; collision cylinder length=0.24 radius=0.02
- link r_hand_pitch: geometry collision box size=0.1 0.05 0.2; visual mesh filename=GR1T2/meshes/r_hand_pitch.STL
- link r_hand_roll: geometry visual mesh filename=GR1T2/meshes/r_hand_roll.STL
- link r_hand_yaw: geometry collision box size=0.065 0.065 0.2; visual mesh filename=GR1T2/meshes/r_hand_yaw.STL
- link r_lower_arm_pitch: geometry visual mesh filename=GR1T2/meshes/r_lower_arm_pitch.STL
- link r_shank_pitch: geometry collision box size=0.07 0.07 0.28; visual mesh filename=GR1T2/meshes/r_shank_pitch.STL
- link r_thigh_pitch: geometry collision box size=0.12 0.08 0.2; collision cylinder length=0.08 radius=0.1
- link r_thigh_roll: geometry visual mesh filename=GR1T2/meshes/r_thigh_roll.STL
- link r_thigh_yaw: geometry collision mesh filename=GR1T2/meshes/r_thigh_yaw.STL; visual mesh filename=GR1T2/meshes/r_thigh_yaw.STL
- link r_upper_arm_pitch: geometry visual mesh filename=GR1T2/meshes/r_upper_arm_pitch.STL
- link r_upper_arm_roll: geometry collision cylinder length=0.08 radius=0.04; visual mesh filename=GR1T2/meshes/r_upper_arm_roll.STL
- link r_upper_arm_yaw: geometry collision cylinder length=0.14 radius=0.035; visual mesh filename=GR1T2/meshes/r_upper_arm_yaw.STL
- link torso: geometry collision mesh filename=GR1T2/meshes/torso.STL; visual mesh filename=GR1T2/meshes/torso.STL
- link waist_pitch: geometry visual mesh filename=GR1T2/meshes/waist_pitch.STL
- link waist_roll: geometry visual mesh filename=GR1T2/meshes/waist_roll.STL
- link waist_yaw: geometry collision mesh filename=GR1T2/meshes/waist_yaw.STL; visual mesh filename=GR1T2/meshes/waist_yaw.STL

File: robot/GRMini1T2/urdf/grmini1t2.urdf (robot description, URDF)
Before this commit: robot GRMini1T2, 46 links, 45 joints
Links:
- link base: geometry collision cylinder length=0.135 radius=0.065; visual mesh filename=GRMini1T2/meshes/base_link.STL
- link camera: geometry visual mesh filename=GRMini1T2/meshes/camera_link.STL
- link imu: geometry visual mesh filename=GRMini1T2/meshes/imu_link.STL
- link left_end_effector: geometry collision sphere radius=0.02751; visual mesh filename=GRMini1T2/meshes/left_end_effector_link.STL
- link left_foot_pitch: geometry collision mesh filename=GRMini1T2/meshes/left_foot_pitch_link.STL; visual mesh filename=GRMini1T2/meshes/left_foot_pitch_link.STL
- link left_foot_roll: geometry visual mesh filename=GRMini1T2/meshes/left_foot_roll_link.STL
- link left_hand_yaw: geometry collision cylinder length=0.12 radius=0.032; visual mesh filename=GRMini1T2/meshes/left_hand_yaw_link.STL
- link left_lower_arm_pitch: geometry visual mesh filename=GRMini1T2/meshes/left_lower_arm_pitch_link.STL
- link left_shank_pitch: geometry collision cylinder length=0.2 radius=0.04; visual mesh filename=GRMini1T2/meshes/left_shank_pitch_link.STL
- link left_thigh_pitch: geometry visual mesh filename=GRMini1T2/meshes/left_thigh_pitch_link.STL
- link left_thigh_roll: geometry collision cylinder length=0.12 radius=0.0415; visual mesh filename=GRMini1T2/meshes/left_thigh_roll_link.STL
- link left_thigh_yaw: geometry collision cylinder length=0.19 radius=0.06; visual mesh filename=GRMini1T2/meshes/left_thigh_yaw_link.STL
- link left_upper_arm_pitch: geometry visual mesh filename=GRMini1T2/meshes/left_upper_arm_pitch_link.STL
- link left_upper_arm_roll: geometry collision sphere radius=0.032; visual mesh filename=GRMini1T2/meshes/left_upper_arm_roll_link.STL
- link left_upper_arm_yaw: geometry collision cylinder length=0.12 radius=0.032; visual mesh filename=GRMini1T2/meshes/left_upper_arm_yaw_link.STL
- link right_end_effector: geometry collision sphere radius=0.02751; visual mesh filename=GRMini1T2/meshes/right_end_effector_link.STL
- link right_foot_pitch: geometry collision mesh filename=GRMini1T2/meshes/right_foot_pitch_link.STL; visual mesh filename=GRMini1T2/meshes/right_foot_pitch_link.STL
- link right_foot_roll: geometry visual mesh filename=GRMini1T2/meshes/right_foot_roll_link.STL
- link right_hand_yaw: geometry collision cylinder length=0.12 radius=0.032; visual mesh filename=GRMini1T2/meshes/right_hand_yaw_link.STL
- link right_lower_arm_pitch: geometry visual mesh filename=GRMini1T2/meshes/right_lower_arm_pitch_link.STL
- link right_shank_pitch: geometry collision cylinder length=0.2 radius=0.04; visual mesh filename=GRMini1T2/meshes/right_shank_pitch_link.STL
- link right_thigh_pitch: geometry visual mesh filename=GRMini1T2/meshes/right_thigh_pitch_link.STL
- link right_thigh_roll: geometry collision cylinder length=0.12 radius=0.0415; visual mesh filename=GRMini1T2/meshes/right_thigh_roll_link.STL
- link right_thigh_yaw: geometry collision cylinder length=0.19 radius=0.06; visual mesh filename=GRMini1T2/meshes/right_thigh_yaw_link.STL
- link right_upper_arm_pitch: geometry visual mesh filename=GRMini1T2/meshes/right_upper_arm_pitch_link.STL
- link right_upper_arm_roll: geometry collision sphere radius=0.032; visual mesh filename=GRMini1T2/meshes/right_upper_arm_roll_link.STL
- link right_upper_arm_yaw: geometry collision cylinder length=0.12 radius=0.032; visual mesh filename=GRMini1T2/meshes/right_upper_arm_yaw_link.STL
- link torso: geometry collision cylinder length=0.22 radius=0.1; collision sphere radius=0.08
- link waist_yaw: geometry collision cylinder length=0.055 radius=0.06; visual mesh filename=GRMini1T2/meshes/waist_yaw_link.STL
Joints:
- joint keyframe_head_joint: origin xyz=0 0 0.28 rpy=0 0 0 -> xyz=0 0 0.18 rpy=0 0 0
- joint keyframe_left_wrist_joint: parent left_hand_pitch -> left_hand_yaw
- joint keyframe_right_wrist_joint: parent right_hand_pitch -> right_hand_yaw
