Commit message: urdf

File: robot/GRMini1T2/urdf/grmini1t2.urdf (robot description, URDF)
Before this commit: robot GRMini1T2, 46 links, 45 joints
Links:
- removed link base_link
- removed link camera_link
- removed link imu_link
- removed link keyframe_head_link
- removed link keyframe_left_ankle_link
- removed link keyframe_left_collar_link
- removed link keyframe_left_elbow_link
- removed link keyframe_left_hip_link
- removed link keyframe_left_knee_link
- removed link keyframe_left_shoulder_link
- removed link keyframe_left_wrist_link
- removed link keyframe_pelvis_link
- removed link keyframe_right_ankle_link
- removed link keyframe_right_collar_link
- removed link keyframe_right_elbow_link
- removed link keyframe_right_hip_link
- removed link keyframe_right_knee_link
- removed link keyframe_right_shoulder_link
- removed link keyframe_right_wrist_link
- removed link keyframe_torso_link
- removed link left_end_effector_link
- removed link left_foot_pitch_link
- removed link left_foot_roll_link
- removed link left_hand_yaw_link
- removed link left_lower_arm_pitch_link
- removed link left_shank_pitch_link
- removed link left_thigh_pitch_link
- removed link left_thigh_roll_link
- removed link left_thigh_yaw_link
- removed link left_upper_arm_pitch_link
- removed link left_upper_arm_roll_link
- removed link left_upper_arm_yaw_link
- removed link right_end_effector_link
- removed link right_foot_pitch_link
- removed link right_foot_roll_link
- removed link right_hand_yaw_link
- removed link right_lower_arm_pitch_link
- removed link right_shank_pitch_link
- removed link right_thigh_pitch_link
- removed link right_thigh_roll_link
- removed link right_thigh_yaw_link
- removed link right_upper_arm_pitch_link
- removed link right_upper_arm_roll_link
- removed link right_upper_arm_yaw_link
- removed link torso_link
- removed link waist_yaw_link
- added link base, mass 3.18; collision cylinder length=0.135 radius=0.065; visual mesh filename=../meshes/base_link.STL
- added link camera, mass 0.0382; visual mesh filename=../meshes/camera_link.STL
- added link imu, mass 0.038; visual mesh filename=../meshes/imu_link.STL
- added link keyframe_head
- added link keyframe_left_ankle
- added link keyframe_left_collar
- added link keyframe_left_elbow
- added link keyframe_left_hip
- added link keyframe_left_knee
- added link keyframe_left_shoulder
- added link keyframe_pelvis
- added link keyframe_right_ankle
- added link keyframe_right_collar
- added link keyframe_right_hip
- added link keyframe_right_knee
- added link keyframe_right_shoulder
- added link keyframe_torso
- added link left_end_effector, mass 0.0994; collision sphere radius=0.02751; visual mesh filename=../meshes/left_end_effector_link.STL
- added link left_foot_pitch, mass 0.528; collision mesh filename=../meshes/left_foot_pitch_link.STL; visual mesh filename=../meshes/left_foot_pitch_link.STL
- added link left_foot_roll, mass 0.113; visual mesh filename=../meshes/left_foot_roll_link.STL
- added link left_hand_yaw, mass 0.440; collision cylinder length=0.12 radius=0.032; visual mesh filename=../meshes/left_hand_yaw_link.STL
- added link left_lower_arm_pitch, mass 0.716; visual mesh filename=../meshes/left_lower_arm_pitch_link.STL
- added link left_shank_pitch, mass 2.21; collision cylinder length=0.2 radius=0.04; visual mesh filename=../meshes/left_shank_pitch_link.STL
- added link left_thigh_pitch, mass 1.31; visual mesh filename=../meshes/left_thigh_pitch_link.STL
- added link left_thigh_roll, mass 1.35; collision cylinder length=0.12 radius=0.0415; visual mesh filename=../meshes/left_thigh_roll_link.STL
- added link left_thigh_yaw, mass 3.37; collision cylinder length=0.19 radius=0.06; visual mesh filename=../meshes/left_thigh_yaw_link.STL
- added link left_upper_arm_pitch, mass 0.885; visual mesh filename=../meshes/left_upper_arm_pitch_link.STL
- added link left_upper_arm_roll, mass 0.716; collision sphere radius=0.032; visual mesh filename=../meshes/left_upper_arm_roll_link.STL
- added link left_upper_arm_yaw, mass 0.913; collision cylinder length=0.12 radius=0.032; visual mesh filename=../meshes/left_upper_arm_yaw_link.STL
- added link right_end_effector, mass 0.0994; collision sphere radius=0.02751; visual mesh filename=../meshes/right_end_effector_link.STL
- added link right_foot_pitch, mass 0.528; collision mesh filename=../meshes/right_foot_pitch_link.STL; visual mesh filename=../meshes/right_foot_pitch_link.STL
- added link right_foot_roll, mass 0.113; visual mesh filename=../meshes/right_foot_roll_link.STL
- added link right_hand_yaw, mass 0.440; collision cylinder length=0.12 radius=0.032; visual mesh filename=../meshes/right_hand_yaw_link.STL
- added link right_lower_arm_pitch, mass 0.716; visual mesh filename=../meshes/right_lower_arm_pitch_link.STL
- added link right_shank_pitch, mass 2.21; collision cylinder length=0.2 radius=0.04; visual mesh filename=../meshes/right_shank_pitch_link.STL
- added link right_thigh_pitch, mass 1.31; visual mesh filename=../meshes/right_thigh_pitch_link.STL
- added link right_thigh_roll, mass 1.35; collision cylinder length=0.12 radius=0.0415; visual mesh filename=../meshes/right_thigh_roll_link.STL
- added link right_thigh_yaw, mass 3.37; collision cylinder length=0.19 radius=0.06; visual mesh filename=../meshes/right_thigh_yaw_link.STL
- added link right_upper_arm_pitch, mass 0.885; visual mesh filename=../meshes/right_upper_arm_pitch_link.STL
- added link right_upper_arm_roll, mass 0.716; collision sphere radius=0.032; visual mesh filename=../meshes/right_upper_arm_roll_link.STL
- added link right_upper_arm_yaw, mass 0.913; collision cylinder length=0.12 radius=0.032; visual mesh filename=../meshes/right_upper_arm_yaw_link.STL
- added link torso, mass 7.99; collision cylinder length=0.22 radius=0.1; collision sphere radius=0.08
- added link waist_yaw, mass 3.18; collision cylinder length=0.055 radius=0.06; visual mesh filename=../meshes/waist_yaw_link.STL
Joints:
- removed joint keyframe_elbow_joint
- removed joint keyframe_left_wrist_joint
- removed joint keyframe_right_wrist_joint
- joint camera_joint: child camera_link -> camera; parent torso_link -> torso
- joint imu_joint: child imu_link -> imu; parent base_link -> base
- joint keyframe_head_joint: child keyframe_head_link -> keyframe_head
- joint keyframe_left_ankle_joint: child keyframe_left_ankle_link -> keyframe_left_ankle; parent l_foot_roll -> left_foot_roll
- joint keyframe_left_collar_joint: child keyframe_left_collar_link -> keyframe_left_collar; parent l_upper_arm_pitch -> left_upper_arm_pitch
- joint keyframe_left_elbow_pitch_joint: child keyframe_left_elbow_link -> keyframe_left_elbow; parent l_lower_arm_pitch -> left_lower_arm_pitch
- joint keyframe_left_hip_joint: child keyframe_left_hip_link -> keyframe_left_hip; parent l_thigh_roll -> left_thigh_roll
- joint keyframe_left_knee_joint: child keyframe_left_knee_link -> keyframe_left_knee; parent l_shank_pitch -> left_shank_pitch
- joint keyframe_left_shoulder_joint: child keyframe_left_shoulder_link -> keyframe_left_shoulder; parent l_upper_arm_roll -> left_upper_arm_roll
- joint keyframe_pelvis_joint: child keyframe_pelvis_link -> keyframe_pelvis
- joint keyframe_right_ankle_joint: child keyframe_right_ankle_link -> keyframe_right_ankle; parent r_foot_roll -> right_foot_roll
- joint keyframe_right_collar_joint: child keyframe_right_collar_link -> keyframe_right_collar; parent r_upper_arm_pitch -> right_upper_arm_pitch
- joint keyframe_right_hip_joint: child keyframe_right_hip_link -> keyframe_right_hip; parent r_thigh_roll -> right_thigh_roll
- joint keyframe_right_knee_joint: child keyframe_right_knee_link -> keyframe_right_knee; parent r_shank_pitch -> right_shank_pitch
- joint keyframe_right_shoulder_joint: child keyframe_right_shoulder_link -> keyframe_right_shoulder; parent r_upper_arm_roll -> right_upper_arm_roll
- joint keyframe_torso_joint: child keyframe_torso_link -> keyframe_torso
- joint left_ankle_pitch_joint: child left_foot_pitch_link -> left_foot_pitch; parent left_foot_roll_link -> left_foot_roll
- joint left_ankle_roll_joint: child left_foot_roll_link -> left_foot_roll; parent left_shank_pitch_link -> left_shank_pitch
- joint left_elbow_pitch_joint: child left_lower_arm_pitch_link -> left_lower_arm_pitch; parent left_upper_arm_yaw_link -> left_upper_arm_yaw
- joint left_end_effector_joint: child left_end_effector_link -> left_end_effector; parent left_hand_yaw_link -> left_hand_yaw
- joint left_hip_pitch_joint: child left_thigh_pitch_link -> left_thigh_pitch; parent base_link -> base
- joint left_hip_roll_joint: child left_thigh_roll_link -> left_thigh_roll; parent left_thigh_pitch_link -> left_thigh_pitch
- joint left_hip_yaw_joint: child left_thigh_yaw_link -> left_thigh_yaw; parent left_thigh_roll_link -> left_thigh_roll
- joint left_knee_pitch_joint: child left_shank_pitch_link -> left_shank_pitch; parent left_thigh_yaw_link -> left_thigh_yaw
- joint left_shoulder_pitch_joint: child left_upper_arm_pitch_link -> left_upper_arm_pitch; parent torso_link -> torso
- joint left_shoulder_roll_joint: child left_upper_arm_roll_link -> left_upper_arm_roll; parent left_upper_arm_pitch_link -> left_upper_arm_pitch
- joint left_shoulder_yaw_joint: child left_upper_arm_yaw_link -> left_upper_arm_yaw; parent left_upper_arm_roll_link -> left_upper_arm_roll
- joint left_wrist_yaw_joint: child left_hand_yaw_link -> left_hand_yaw; parent left_lower_arm_pitch_link -> left_lower_arm_pitch
- joint right_ankle_pitch_joint: child right_foot_pitch_link -> right_foot_pitch; parent right_foot_roll_link -> right_foot_roll
- joint right_ankle_roll_joint: child right_foot_roll_link -> right_foot_roll; parent right_shank_pitch_link -> right_shank_pitch
- joint right_elbow_pitch_joint: child right_lower_arm_pitch_link -> right_lower_arm_pitch; parent right_upper_arm_yaw_link -> right_upper_arm_yaw
- joint right_end_effector_joint: child right_end_effector_link -> right_end_effector; parent right_hand_yaw_link -> right_hand_yaw
- joint right_hip_pitch_joint: child right_thigh_pitch_link -> right_thigh_pitch; parent base_link -> base
- joint right_hip_roll_joint: child right_thigh_roll_link -> right_thigh_roll; parent right_thigh_pitch_link -> right_thigh_pitch
- joint right_hip_yaw_joint: child right_thigh_yaw_link -> right_thigh_yaw; parent right_thigh_roll_link -> right_thigh_roll
- joint right_knee_pitch_joint: child right_shank_pitch_link -> right_shank_pitch; parent right_thigh_yaw_link -> right_thigh_yaw
- joint right_shoulder_pitch_joint: child right_upper_arm_pitch_link -> right_upper_arm_pitch; parent torso_link -> torso
- joint right_shoulder_roll_joint: child right_upper_arm_roll_link -> right_upper_arm_roll; parent right_upper_arm_pitch_link -> right_upper_arm_pitch
- joint right_shoulder_yaw_joint: child right_upper_arm_yaw_link -> right_upper_arm_yaw; parent right_upper_arm_roll_link -> right_upper_arm_roll
- joint right_wrist_yaw_joint: child right_hand_yaw_link -> right_hand_yaw; parent right_lower_arm_pitch_link -> right_lower_arm_pitch
- joint torso_joint: child torso_link -> torso; parent waist_yaw_link -> waist_yaw
- joint waist_yaw_joint: child waist_yaw_link -> waist_yaw; parent base_link -> base

Commit message: urdf mapping

File: robot/GRMini1T2/urdf/grmini1t2.urdf (robot description, URDF)
Before this commit: robot GRMini1T2, 43 links, 42 joints
Links:
- added link keyframe_left_wrist
- added link keyframe_right_elbow
- added link keyframe_right_wrist
Joints:
- added joint keyframe_elbow_joint: type fixed, parent right_lower_arm_pitch, child keyframe_right_elbow, origin xyz=0 0 0 rpy=0 0 0
- added joint keyframe_left_wrist_joint: type fixed, parent left_hand_pitch, child keyframe_left_wrist, origin xyz=0 0 -0.1 rpy=0 0 0
- added joint keyframe_right_wrist_joint: type fixed, parent right_hand_pitch, child keyframe_right_wrist, origin xyz=0 0 -0.1 rpy=0 0 0

Commit message: finished

File: robot/GRMini1T2/urdf/grmini1t2.urdf (robot description, URDF)
Before this commit: robot GRMini1T2, 46 links, 45 joints
Links:
- removed link keyframe_head
- removed link keyframe_left_ankle
- removed link keyframe_left_collar
- removed link keyframe_left_elbow
- removed link keyframe_left_hip
- removed link keyframe_left_knee
- removed link keyframe_left_shoulder
- removed link keyframe_left_wrist
- removed link keyframe_pelvis
- removed link keyframe_right_ankle
- removed link keyframe_right_collar
- removed link keyframe_right_elbow
- removed link keyframe_right_hip
- removed link keyframe_right_knee
- removed link keyframe_right_shoulder
- removed link keyframe_right_wrist
- removed link keyframe_torso
- added link keyframe_head_link
- added link keyframe_left_ankle_link
- added link keyframe_left_collar_link
- added link keyframe_left_elbow_link
- added link keyframe_left_hip_link
- added link keyframe_left_knee_link
- added link keyframe_left_shoulder_link
- added link keyframe_left_wrist_link
- added link keyframe_pelvis_link
- added link keyframe_right_ankle_link
- added link keyframe_right_collar_link
- added link keyframe_right_elbow_link
- added link keyframe_right_hip_link
- added link keyframe_right_knee_link
- added link keyframe_right_shoulder_link
- added link keyframe_right_wrist_link
- added link keyframe_torso_link
Joints:
- joint keyframe_elbow_joint: child keyframe_right_elbow -> keyframe_right_elbow_link
- joint keyframe_head_joint: child keyframe_head -> keyframe_head_link
- joint keyframe_left_ankle_joint: child keyframe_left_ankle -> keyframe_left_ankle_link
- joint keyframe_left_collar_joint: child keyframe_left_collar -> keyframe_left_collar_link
- joint keyframe_left_elbow_pitch_joint: child keyframe_left_elbow -> keyframe_left_elbow_link
- joint keyframe_left_hip_joint: child keyframe_left_hip -> keyframe_left_hip_link
- joint keyframe_left_knee_joint: child keyframe_left_knee -> keyframe_left_knee_link
- joint keyframe_left_shoulder_joint: child keyframe_left_shoulder -> keyframe_left_shoulder_link
- joint keyframe_left_wrist_joint: child keyframe_left_wrist -> keyframe_left_wrist_link
- joint keyframe_pelvis_joint: child keyframe_pelvis -> keyframe_pelvis_link
- joint keyframe_right_ankle_joint: child keyframe_right_ankle -> keyframe_right_ankle_link
- joint keyframe_right_collar_joint: child keyframe_right_collar -> keyframe_right_collar_link
- joint keyframe_right_hip_joint: child keyframe_right_hip -> keyframe_right_hip_link
- joint keyframe_right_knee_joint: child keyframe_right_knee -> keyframe_right_knee_link
- joint keyframe_right_shoulder_joint: child keyframe_right_shoulder -> keyframe_right_shoulder_link
- joint keyframe_right_wrist_joint: child keyframe_right_wrist -> keyframe_right_wrist_link
- joint keyframe_torso_joint: child keyframe_torso -> keyframe_torso_link
