Commit message: modified grmini1t2

File: robot/G1/urdf/g1.urdf (robot description, URDF)
Before this commit: robot g1, 48 links, 47 joints
Links:
- link head_link: geometry collision mesh filename=../../G1/meshes/head_link.STL; visual mesh filename=../../G1/meshes/head_link.STL
- link left_ankle_pitch_link: geometry collision mesh filename=../../G1/meshes/left_ankle_pitch_link.STL; visual mesh filename=../../G1/meshes/left_ankle_pitch_link.STL
- link left_ankle_roll_link: geometry collision sphere radius=0.005; collision sphere radius=0.005
- link left_elbow_link: geometry collision mesh filename=../../G1/meshes/left_elbow_link.STL; visual mesh filename=../../G1/meshes/left_elbow_link.STL
- link left_hip_pitch_link: geometry collision mesh filename=../../G1/meshes/left_hip_pitch_link.STL; visual mesh filename=../../G1/meshes/left_hip_pitch_link.STL
- link left_hip_roll_link: geometry collision mesh filename=../../G1/meshes/left_hip_roll_link.STL; visual mesh filename=../../G1/meshes/left_hip_roll_link.STL
- link left_hip_yaw_link: geometry collision mesh filename=../../G1/meshes/left_hip_yaw_link.STL; visual mesh filename=../../G1/meshes/left_hip_yaw_link.STL
- link left_knee_link: geometry collision mesh filename=../../G1/meshes/left_knee_link.STL; visual mesh filename=../../G1/meshes/left_knee_link.STL
- link left_shoulder_pitch_link: geometry collision cylinder length=0.05 radius=0.03; visual mesh filename=../../G1/meshes/left_shoulder_pitch_link.STL
- link left_shoulder_roll_link: geometry collision cylinder length=0.03 radius=0.03; visual mesh filename=../../G1/meshes/left_shoulder_roll_link.STL
- link left_shoulder_yaw_link: geometry collision mesh filename=../../G1/meshes/left_shoulder_yaw_link.STL; visual mesh filename=../../G1/meshes/left_shoulder_yaw_link.STL
- link left_wrist_roll_rubber_hand: geometry collision mesh filename=../../G1/meshes/left_wrist_roll_rubber_hand.STL; visual mesh filename=../../G1/meshes/left_wrist_roll_rubber_hand.STL
- link logo_link: geometry collision mesh filename=../../G1/meshes/logo_link.STL; visual mesh filename=../../G1/meshes/logo_link.STL
- link pelvis: geometry visual mesh filename=../../G1/meshes/pelvis.STL
- link pelvis_contour_link: geometry collision mesh filename=../../G1/meshes/pelvis_contour_link.STL; visual mesh filename=../../G1/meshes/pelvis_contour_link.STL
- link right_ankle_pitch_link: geometry collision mesh filename=../../G1/meshes/right_ankle_pitch_link.STL; visual mesh filename=../../G1/meshes/right_ankle_pitch_link.STL
- link right_ankle_roll_link: geometry collision sphere radius=0.005; collision sphere radius=0.005
- link right_elbow_link: geometry collision mesh filename=../../G1/meshes/right_elbow_link.STL; visual mesh filename=../../G1/meshes/right_elbow_link.STL
- link right_hip_pitch_link: geometry collision mesh filename=../../G1/meshes/right_hip_pitch_link.STL; visual mesh filename=../../G1/meshes/right_hip_pitch_link.STL
- link right_hip_roll_link: geometry collision mesh filename=../../G1/meshes/right_hip_roll_link.STL; visual mesh filename=../../G1/meshes/right_hip_roll_link.STL
- link right_hip_yaw_link: geometry collision mesh filename=../../G1/meshes/right_hip_yaw_link.STL; visual mesh filename=../../G1/meshes/right_hip_yaw_link.STL
- link right_knee_link: geometry collision mesh filename=../../G1/meshes/right_knee_link.STL; visual mesh filename=../../G1/meshes/right_knee_link.STL
- link right_shoulder_pitch_link: geometry collision cylinder length=0.05 radius=0.03; visual mesh filename=../../G1/meshes/right_shoulder_pitch_link.STL
- link right_shoulder_roll_link: geometry collision cylinder length=0.03 radius=0.03; visual mesh filename=../../G1/meshes/right_shoulder_roll_link.STL
- link right_shoulder_yaw_link: geometry collision mesh filename=../../G1/meshes/right_shoulder_yaw_link.STL; visual mesh filename=../../G1/meshes/right_shoulder_yaw_link.STL
- link right_wrist_roll_rubber_hand: geometry collision mesh filename=../../G1/meshes/right_wrist_roll_rubber_hand.STL; visual mesh filename=../../G1/meshes/right_wrist_roll_rubber_hand.STL
- link torso_link: geometry collision mesh filename=../../G1/meshes/torso_link_23dof_rev_1_0.STL; visual mesh filename=../../G1/meshes/torso_link_23dof_rev_1_0.STL

File: robot/GR1T2/urdf/gr1t2.urdf (robot description, URDF)
Before this commit: robot GR1T2, 51 links, 50 joints
Links:
- link base: geometry collision mesh filename=../../GR1T2/meshes/base.STL; visual mesh filename=../../GR1T2/meshes/base.STL
- link head_pitch: geometry visual mesh filename=../../GR1T2/meshes/head_pitch.STL
- link head_roll: geometry visual mesh filename=../../GR1T2/meshes/head_roll.STL
- link head_yaw: geometry collision sphere radius=0.12; visual mesh filename=../../GR1T2/meshes/head_yaw.STL
- link l_foot_pitch: geometry visual mesh filename=../../GR1T2/meshes/l_foot_pitch.STL
- link l_foot_roll: geometry collision cylinder length=0.24 radius=0.02; collision cylinder length=0.24 radius=0.02
- link l_hand_pitch: geometry collision box size=0.1 0.05 0.2; visual mesh filename=../../GR1T2/meshes/l_hand_pitch.STL
- link l_hand_roll: geometry visual mesh filename=../../GR1T2/meshes/l_hand_roll.STL
- link l_hand_yaw: geometry collision box size=0.065 0.065 0.2; visual mesh filename=../../GR1T2/meshes/l_hand_yaw.STL
- link l_lower_arm_pitch: geometry visual mesh filename=../../GR1T2/meshes/l_lower_arm_pitch.STL
- link l_shank_pitch: geometry collision box size=0.07 0.07 0.28; visual mesh filename=../../GR1T2/meshes/l_shank_pitch.STL
- link l_thigh_pitch: geometry collision box size=0.12 0.08 0.2; collision cylinder length=0.08 radius=0.1
- link l_thigh_roll: geometry visual mesh filename=../../GR1T2/meshes/l_thigh_roll.STL
- link l_thigh_yaw: geometry collision mesh filename=../../GR1T2/meshes/l_thigh_yaw.STL; visual mesh filename=../../GR1T2/meshes/l_thigh_yaw.STL
- link l_upper_arm_pitch: geometry visual mesh filename=../../GR1T2/meshes/l_upper_arm_pitch.STL
- link l_upper_arm_roll: geometry collision cylinder length=0.08 radius=0.04; visual mesh filename=../../GR1T2/meshes/l_upper_arm_roll.STL
- link l_upper_arm_yaw: geometry collision cylinder length=0.14 radius=0.035; visual mesh filename=../../GR1T2/meshes/l_upper_arm_yaw.STL
- link r_foot_pitch: geometry visual mesh filename=../../GR1T2/meshes/r_foot_pitch.STL
- link r_foot_roll: geometry collision cylinder length=0.24 radius=0.02; collision cylinder length=0.24 radius=0.02
- link r_hand_pitch: geometry collision box size=0.1 0.05 0.2; visual mesh filename=../../GR1T2/meshes/r_hand_pitch.STL
- link r_hand_roll: geometry visual mesh filename=../../GR1T2/meshes/r_hand_roll.STL
- link r_hand_yaw: geometry collision box size=0.065 0.065 0.2; visual mesh filename=../../GR1T2/meshes/r_hand_yaw.STL
- link r_lower_arm_pitch: geometry visual mesh filename=../../GR1T2/meshes/r_lower_arm_pitch.STL
- link r_shank_pitch: geometry collision box size=0.07 0.07 0.28; visual mesh filename=../../GR1T2/meshes/r_shank_pitch.STL
- link r_thigh_pitch: geometry collision box size=0.12 0.08 0.2; collision cylinder length=0.08 radius=0.1
- link r_thigh_roll: geometry visual mesh filename=../../GR1T2/meshes/r_thigh_roll.STL
- link r_thigh_yaw: geometry collision mesh filename=../../GR1T2/meshes/r_thigh_yaw.STL; visual mesh filename=../../GR1T2/meshes/r_thigh_yaw.STL
- link r_upper_arm_pitch: geometry visual mesh filename=../../GR1T2/meshes/r_upper_arm_pitch.STL
- link r_upper_arm_roll: geometry collision cylinder length=0.08 radius=0.04; visual mesh filename=../../GR1T2/meshes/r_upper_arm_roll.STL
- link r_upper_arm_yaw: geometry collision cylinder length=0.14 radius=0.035; visual mesh filename=../../GR1T2/meshes/r_upper_arm_yaw.STL
- link torso: geometry collision mesh filename=../../GR1T2/meshes/torso.STL; visual mesh filename=../../GR1T2/meshes/torso.STL
- link waist_pitch: geometry visual mesh filename=../../GR1T2/meshes/waist_pitch.STL
- link waist_roll: geometry visual mesh filename=../../GR1T2/meshes/waist_roll.STL
- link waist_yaw: geometry collision mesh filename=../../GR1T2/meshes/waist_yaw.STL; visual mesh filename=../../GR1T2/meshes/waist_yaw.STL

File: robot/GRMini1T2/urdf/grmini1t2.urdf (robot description, URDF)
Before this commit: robot GRMini1T2, 29 links, 28 joints
Links:
- added link keyframe_head_link
- added link keyframe_left_ankle_link
- added link keyframe_left_collar_link
- added link keyframe_left_elbow_link
- added link keyframe_left_hip_link
- added link keyframe_left_knee_link
- added link keyframe_left_shoulder_link
- added link keyframe_left_wrist_link
- added link keyframe_pelvis_link
- added link keyframe_right_ankle_link
- added link keyframe_right_collar_link
- added link keyframe_right_elbow_link
- added link keyframe_right_hip_link
- added link keyframe_right_knee_link
- added link keyframe_right_shoulder_link
- added link keyframe_right_wrist_link
- added link keyframe_torso_link
Joints:
- added joint keyframe_elbow_joint: type fixed, parent r_lower_arm_pitch, child keyframe_right_elbow_link, origin xyz=0 0 0 rpy=0 0 0
- added joint keyframe_head_joint: type fixed, parent torso, child keyframe_head_link, origin xyz=0 0 0.28 rpy=0 0 0
- added joint keyframe_left_ankle_joint: type fixed, parent l_foot_roll, child keyframe_left_ankle_link, origin xyz=0 0 0 rpy=0 0 0
- added joint keyframe_left_collar_joint: type fixed, parent l_upper_arm_pitch, child keyframe_left_collar_link, origin xyz=0 0 0.04 rpy=0 0 0
- added joint keyframe_left_elbow_pitch_joint: type fixed, parent l_lower_arm_pitch, child keyframe_left_elbow_link, origin xyz=0 0 0 rpy=0 0 0
- added joint keyframe_left_hip_joint: type fixed, parent l_thigh_roll, child keyframe_left_hip_link, origin xyz=0 0 0 rpy=0 0 0
- added joint keyframe_left_knee_joint: type fixed, parent l_shank_pitch, child keyframe_left_knee_link, origin xyz=0 0 0 rpy=0 0 0
- added joint keyframe_left_shoulder_joint: type fixed, parent l_upper_arm_roll, child keyframe_left_shoulder_link, origin xyz=0 0 0 rpy=0 0 0
- added joint keyframe_left_wrist_joint: type fixed, parent l_hand_pitch, child keyframe_left_wrist_link, origin xyz=0 0 -0.1 rpy=0 0 0
- added joint keyframe_pelvis_joint: type fixed, parent base, child keyframe_pelvis_link, origin xyz=0 0 0 rpy=0 0 0
- added joint keyframe_right_ankle_joint: type fixed, parent r_foot_roll, child keyframe_right_ankle_link, origin xyz=0 0 0 rpy=0 0 0
- added joint keyframe_right_collar_joint: type fixed, parent r_upper_arm_pitch, child keyframe_right_collar_link, origin xyz=0 0 0.04 rpy=0 0 0
- added joint keyframe_right_hip_joint: type fixed, parent r_thigh_roll, child keyframe_right_hip_link, origin xyz=0 0 0 rpy=0 0 0
- added joint keyframe_right_knee_joint: type fixed, parent r_shank_pitch, child keyframe_right_knee_link, origin xyz=0 0 0 rpy=0 0 0
- added joint keyframe_right_shoulder_joint: type fixed, parent r_upper_arm_roll, child keyframe_right_shoulder_link, origin xyz=0 0 0 rpy=0 0 0
- added joint keyframe_right_wrist_joint: type fixed, parent r_hand_pitch, child keyframe_right_wrist_link, origin xyz=0 0 -0.1 rpy=0 0 0
- added joint keyframe_torso_joint: type fixed, parent torso, child keyframe_torso_link, origin xyz=0 0 0 rpy=0 0 0

Commit message: 1

File: robot/G1/urdf/g1.urdf (robot description, URDF)
Before this commit: robot ../../G1, 48 links, 47 joints
Links:
- link head_link: geometry collision mesh filename=G1/meshes/head_link.STL; visual mesh filename=G1/meshes/head_link.STL
- link left_ankle_pitch_link: geometry collision mesh filename=G1/meshes/left_ankle_pitch_link.STL; visual mesh filename=G1/meshes/left_ankle_pitch_link.STL
- link left_ankle_roll_link: geometry collision sphere radius=0.005; collision sphere radius=0.005
- link left_elbow_link: geometry collision mesh filename=G1/meshes/left_elbow_link.STL; visual mesh filename=G1/meshes/left_elbow_link.STL
- link left_hip_pitch_link: geometry collision mesh filename=G1/meshes/left_hip_pitch_link.STL; visual mesh filename=G1/meshes/left_hip_pitch_link.STL
- link left_hip_roll_link: geometry collision mesh filename=G1/meshes/left_hip_roll_link.STL; visual mesh filename=G1/meshes/left_hip_roll_link.STL
- link left_hip_yaw_link: geometry collision mesh filename=G1/meshes/left_hip_yaw_link.STL; visual mesh filename=G1/meshes/left_hip_yaw_link.STL
- link left_knee_link: geometry collision mesh filename=G1/meshes/left_knee_link.STL; visual mesh filename=G1/meshes/left_knee_link.STL
- link left_shoulder_pitch_link: geometry collision cylinder length=0.05 radius=0.03; visual mesh filename=G1/meshes/left_shoulder_pitch_link.STL
- link left_shoulder_roll_link: geometry collision cylinder length=0.03 radius=0.03; visual mesh filename=G1/meshes/left_shoulder_roll_link.STL
- link left_shoulder_yaw_link: geometry collision mesh filename=G1/meshes/left_shoulder_yaw_link.STL; visual mesh filename=G1/meshes/left_shoulder_yaw_link.STL
- link left_wrist_roll_rubber_hand: geometry collision mesh filename=G1/meshes/left_wrist_roll_rubber_hand.STL; visual mesh filename=G1/meshes/left_wrist_roll_rubber_hand.STL
- link logo_link: geometry collision mesh filename=G1/meshes/logo_link.STL; visual mesh filename=G1/meshes/logo_link.STL
- link pelvis: geometry visual mesh filename=G1/meshes/pelvis.STL
- link pelvis_contour_link: geometry collision mesh filename=G1/meshes/pelvis_contour_link.STL; visual mesh filename=G1/meshes/pelvis_contour_link.STL
- link right_ankle_pitch_link: geometry collision mesh filename=G1/meshes/right_ankle_pitch_link.STL; visual mesh filename=G1/meshes/right_ankle_pitch_link.STL
- link right_ankle_roll_link: geometry collision sphere radius=0.005; collision sphere radius=0.005
- link right_elbow_link: geometry collision mesh filename=G1/meshes/right_elbow_link.STL; visual mesh filename=G1/meshes/right_elbow_link.STL
- link right_hip_pitch_link: geometry collision mesh filename=G1/meshes/right_hip_pitch_link.STL; visual mesh filename=G1/meshes/right_hip_pitch_link.STL
- link right_hip_roll_link: geometry collision mesh filename=G1/meshes/right_hip_roll_link.STL; visual mesh filename=G1/meshes/right_hip_roll_link.STL
- link right_hip_yaw_link: geometry collision mesh filename=G1/meshes/right_hip_yaw_link.STL; visual mesh filename=G1/meshes/right_hip_yaw_link.STL
- link right_knee_link: geometry collision mesh filename=G1/meshes/right_knee_link.STL; visual mesh filename=G1/meshes/right_knee_link.STL
- link right_shoulder_pitch_link: geometry collision cylinder length=0.05 radius=0.03; visual mesh filename=G1/meshes/right_shoulder_pitch_link.STL
- link right_shoulder_roll_link: geometry collision cylinder length=0.03 radius=0.03; visual mesh filename=G1/meshes/right_shoulder_roll_link.STL
- link right_shoulder_yaw_link: geometry collision mesh filename=G1/meshes/right_shoulder_yaw_link.STL; visual mesh filename=G1/meshes/right_shoulder_yaw_link.STL
- link right_wrist_roll_rubber_hand: geometry collision mesh filename=G1/meshes/right_wrist_roll_rubber_hand.STL; visual mesh filename=G1/meshes/right_wrist_roll_rubber_hand.STL
- link torso_link: geometry collision mesh filename=G1/meshes/torso_link_23dof_rev_1_0.STL; visual mesh filename=G1/meshes/torso_link_23dof_rev_1_0.STL
