Commit message: 1

File: robot/Ball/Ball.urdf (robot description, URDF)
Before this commit: robot sphere, 1 links, 0 joints
Links:
- removed link base_link
- added link ball_base_link, mass 1.0; collision sphere radius=0.1; visual sphere radius=0.1
- added link ball_tip_link, mass 0.5; collision sphere radius=0.1; visual sphere radius=0.1
Joints:
- added joint ball_joint: type revolute, parent ball_base_link, child ball_tip_link, origin xyz=0 0 1 rpy=0 0 0, axis 0 0 1, limit lower=-3.14 upper=3.14 effort=10 velocity=1
